File: Hardware/Schematic/NixieClock.sch (KiCad schematic (older format))
At the start: 11 parts

Commit message: Converted schematic to a multisheet solution
Parts:
- removed H? (x4): IN-16, ~, symbol IN-16
- removed U? (x4): 74141, ~, symbol 74141
- gave numbers to parts that had none: 3
Connections:
- net labels added: GND, VCC
- wire segments 0 -> 41
- no-connect marks 0 -> 1
Other:
- moved on the sheet: IC101, U101, U102
